Commit message: modify model

File: urdf/dobot.urdf (robot description, URDF)
Before this commit: robot dobot_arm, 5 links, 4 joints
Links:
- added link base_dummy_link; visual box size=0 0 0
- added link fake_link, mass 1; collision box size=0.08 0.03 0.03; visual box size=0.08 0.03 0.03
- added link stick_link, mass 1; collision cylinder length=0.07 radius=0.0055; visual cylinder length=0.07 radius=0.0055
- link chuck_link: geometry collision cylinder length=0.07 radius=0.01; visual cylinder length=0.07 radius=0.01
Joints:
- added joint base_dummy_joint: type fixed, parent base_dummy_link, child base_link, origin xyz=0 0 0 rpy=0 0 0, axis 0 0 0
- added joint fake_joint: type revolute, parent forearm_link, child fake_link, origin xyz=0 0 0.147 rpy=0 0 0, axis 0 1 0, limit lower=-2.8707963267948966 upper=0.2707963267948966 effort=300 velocity=1
- added joint stick_joint: type fixed, parent chuck_link, child stick_link, origin xyz=0 0 -0.11 rpy=0 0.5 0, axis 0 0 0, limit lower=0 upper=0 effort=0 velocity=1
- joint chuck_joint: axis 0 1 0 -> 0 0 1; limit lower=-1.5707963267948966 upper=1.5707963267948966 effort=300 velocity=1 -> lower=-3 upper=3 effort=10 velocity=1; origin xyz=0 0 0.147 rpy=0 0 0 -> xyz=0.05 0 0.0405 rpy=0 0 0; parent forearm_link -> fake_link
- joint forearm_joint: limit lower=-0.1745329251994329577 upper=1.65806278939 effort=300 velocity=1 -> lower=-0.7745329251994329577 upper=1.05806278939 effort=300 velocity=1

Commit message: Update dobot model

File: urdf/dobot.urdf (robot description, URDF)
Before this commit: robot dobot_arm, 8 links, 7 joints
Links:
- link bigarm_link: geometry collision cylinder length=0.2 radius=0.03; visual cylinder length=0.2 radius=0.03
- link forearm_link: geometry collision cylinder length=0.21 radius=0.03; visual cylinder length=0.21 radius=0.03
- link shoulder_link: geometry collision cylinder length=0.065 radius=0.06; visual cylinder length=0.065 radius=0.06
Joints:
- joint bigarm_joint: origin xyz=0 0 0.085 rpy=0 0 0 -> xyz=0 0 0.109 rpy=0 0 0
- joint chuck_joint: limit lower=-3 upper=3 effort=10 velocity=1 -> lower=-2.36 upper=2.36 effort=10 velocity=1
- joint fake_joint: origin xyz=0 0 0.147 rpy=0 0 0 -> xyz=0 0 0.21 rpy=0 0 0
- joint forearm_joint: limit lower=-0.7745329251994329577 upper=1.05806278939 effort=300 velocity=1 -> lower=0.2707963267948966 upper=2.8707963267948966 effort=300 velocity=1; origin xyz=0 0 0.135 rpy=0 0 0 -> xyz=0.015 0 0.14 rpy=0 0 0
- joint shoulder_joint: origin xyz=0 0 0.055 rpy=0 0 0 -> xyz=0 0 0.0425 rpy=0 0 0
