Commit message: attempting inverse kinematics

File: urdf/abb.urdf (robot description, URDF)
Before this commit: robot abb_arm, 8 links, 7 joints
Links:
- removed link chuck_link
- removed link gripper_link
- removed link left_finger_link
- added link elbow_link, mass .1; collision cylinder length=0.02 radius=0.02; visual cylinder length=0.02 radius=0.02
- added link endeffector, mass .1; collision box size=0.08 0.005 0.005; visual box size=0.08 0.005 0.005
- added link hand_link, mass .1; collision box size=0.02 0.01 0.03; visual box size=0.02 0.01 0.03
- link base_dummy_link: mass None -> .5; geometry collision box size=0 0 0; visual box size=0 0 0
- link base_link: mass 1 -> .5; geometry collision box size=0.095 0.077 0.02; visual box size=0.095 0.077 0.02
- link bigarm_link: mass 1 -> .1; geometry collision box size=0.04 0.04 0.13; visual box size=0.04 0.04 0.13
- link forearm_link: mass 1 -> .1; geometry collision box size=0.025 0.025 0.16; visual box size=0.025 0.025 0.16
- link shoulder_link: mass 1 -> .1; geometry collision box size=0.12 0.06 0.05; visual box size=0.12 0.06 0.05
Joints:
- removed joint chuck_joint
- removed joint gripper_joint
- added joint elbow_joint: type revolute, parent bigarm_link, child elbow_link, origin xyz=0 0 0.13 rpy=0 0 0, axis 0 1 0, limit lower=0.785 upper=2.356 effort=300 velocity=1
- added joint endeff_joint: type revolute, parent hand_link, child endeffector, origin xyz=0 0 0.03 rpy=0 0 0, axis 0 0 1, limit lower=-2.094 upper=2.094 effort=10 velocity=1
- joint bigarm_joint: limit lower=-1.483529864195 upper=1.483529864195 effort=300 velocity=1 -> lower=-1.48353 upper=1.48353 effort=300 velocity=1; origin xyz=0 0 0.065 rpy=0 0 0 -> xyz=0.04 0 0.05 rpy=0 0 0
- joint forearm_joint: axis 0 1 0 -> 0 0 1; limit lower=0.2707963267948966 upper=2.8707963267948966 effort=300 velocity=1 -> lower=-2.094 upper=2.094 effort=300 velocity=1; origin xyz=0.0 0 0.145 rpy=0 0 0 -> xyz=0 0 0.02 rpy=0 0 0; parent bigarm_link -> elbow_link
- joint hand_joint: axis 1 0 0 -> 0 1 0; child left_finger_link -> hand_link; limit lower=-2.36 upper=2.36 effort=10 velocity=1 -> lower=-2.094 upper=2.094 effort=10 velocity=1; origin xyz=0 0 -0.057 rpy=0 0 0 -> xyz=0 0 0.16 rpy=0 0 0; parent chuck_link -> forearm_link
- joint shoulder_joint: limit lower=-2.35619449 upper=2.35619449 effort=300 velocity=1 -> lower=-2.094 upper=2.094 effort=300 velocity=1; origin xyz=0 0 0.015 rpy=0 0 0 -> xyz=0 0 0.03 rpy=0 0 0

Commit message: attempting ik

File: urdf/abb.urdf (robot description, URDF)
Before this commit: robot abb_arm, 8 links, 7 joints
Joints:
- joint base_dummy_joint: origin xyz=0 0 0 rpy=0 0 0 -> xyz=-0.25 0 0 rpy=0 0 0
